File: peripherals.kicad_sch (KiCad schematic)
At the start: 5 parts, among them J5 Micro_SD_Card_Det2

Commit message: Add in LCSC part numbers for major parts, assign packages
Parts:
- C63, C64, C65: footprint (none) -> Capacitor_SMD:C_0402_1005Metric
- J5: LCSC Part # (none) -> C114218
- U1: LCSC Part # (none) -> C414042
Changed lines of the file:
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@@
 			)
 		)
-		(property "Footprint" ""
+		(property "Footprint" "Capacitor_SMD:C_0402_1005Metric"
 			(at 30.7848 43.18 0)
 			(effects
@@
 			)
 		)
+		(property "LCSC Part #" "C414042"
+			(at 167.64 118.11 0)
+			(effects
+				(font
+					(size 1.27 1.27)
+				)
+				(hide yes)
+			)
+		)
 		(pin "A6"
 		)
@@
 			)
 		)
+		(property "LCSC Part #" "C414042"
+			(at 55.88 40.64 0)
+			(effects
+				(font
+					(size 1.27 1.27)
+				)
+				(hide yes)
+			)
+		)
 		(pin "A6"
 		)
@@
 			)
 		)
+		(property "LCSC Part #" "C414042"
+			(at 59.69 69.85 0)
+			(effects
+				(font
+					(size 1.27 1.27)
+				)
+				(hide yes)
+			)
+		)
 		(pin "A6"
 		)
@@
 			)
 		)
-		(property "Footprint" ""
+		(property "Footprint" "Capacitor_SMD:C_0402_1005Metric"
 			(at 38.4048 111.76 0)
 			(effects
@@
 			)
 		)
+		(property "LCSC Part #" "C414042"
+			(at 69.85 114.3 0)
+			(effects
+				(font
+					(size 1.27 1.27)
+				)
+				(hide yes)
+			)
+		)
 		(pin "A6"
 		)
@@
 			)
 		)
+		(property "LCSC Part #" "C114218"
+			(at 125.73 43.18 0)
+			(effects
+				(font
+					(size 1.27 1.27)
+				)
+				(hide yes)
+			)
+		)
 		(pin "5"
 		)
@@
 			)
 		)
-		(property "Footprint" ""
+		(property "Footprint" "Capacitor_SMD:C_0402_1005Metric"
 			(at 143.8148 110.49 0)
 			(effects
