File: imx6test.kicad_pcb (KiCad board)
At the start: 4 copper layers, 100 x 75 mm, 163 parts, among them J1 Barrel_Jack_MountingPin, J2 Conn_ARM_JTAG_SWD_20, J3 Conn_01x06_Pin, J4 Conn_01x06_Pin, J5 Micro_SD_Card_Det2, J6 USB_A, SW1 SW_DIP_x04, SW3 SW_SPST, Y1 32.768k, Y2 24MHz

Commit message: Small update
Parts:
- R53, R58: moved to B.Cu
- moved U9 170.7 mm to (110.5, 86.5)
- moved Q1 144.3 mm to (115.8, 96.0)
- moved Q2 144.3 mm to (112.0, 92.5)
- moved Q3 144.3 mm to (112.0, 96.4)
- moved U2 144.3 mm to (116.1, 92.5)
- moved U5 143.1 mm to (111.0, 80.0)
- moved U4 136.9 mm to (116.5, 80.0)
- moved U3 134.8 mm to (117.0, 87.0)
- moved R58 60.3 mm to (192.0, 59.0), turned to 180 degrees
- moved R53 57.5 mm to (194.0, 59.0), turned to 180 degrees
- moved C1 0.83 mm to (220.2, 118.0)
Routing:
- added copper zone on B.Cu, net GND
- removed copper zone on F.Cu, net GND
